File: hardware/extension.r0/extension.r0.kicad_pcb (KiCad board)
At the start: 2 copper layers, 5 parts, among them J1 JTAG, J2 UART

Commit message: backup
Parts:
- added Debug1: Conn_02x07_Odd_Even, Connector_IDC:IDC-Header_2x07_P2.54mm_Horizontal, F.Cu at (77.2, 119.9)
- added J7: Vdrive_I, Connector_PinHeader_2.54mm:PinHeader_1x01_P2.54mm_Vertical, B.Cu at (93.0, 74.2)
- added Logic1: Conn_02x10_Odd_Even, Connector_IDC:IDC-Header_2x10_P2.54mm_Horizontal, F.Cu at (114.3, 119.9)
- added POWER1: Conn_01x01, Connector_PinSocket_2.54mm:PinSocket_1x01_P2.54mm_Vertical, B.Cu at (112.7, 77.9)
- added ULPI1: Conn_01x01, Connector_PinSocket_2.00mm:PinSocket_1x01_P2.00mm_Vertical, B.Cu at (106.3, 80.4)
- added ULPI11: Conn_01x01, Connector_PinSocket_2.00mm:PinSocket_1x01_P2.00mm_Vertical, B.Cu at (59.4, 87.0)
- added ULPI12: Conn_01x01, Connector_PinSocket_2.00mm:PinSocket_1x01_P2.00mm_Vertical, B.Cu at (93.0, 86.0)
- added ULPI2: Conn_01x01, Connector_PinSocket_2.00mm:PinSocket_1x01_P2.00mm_Vertical, B.Cu at (102.1, 79.0)
- added ULPI3: Conn_01x01, Connector_PinSocket_2.00mm:PinSocket_1x01_P2.00mm_Vertical, B.Cu at (58.4, 77.6)
- added ULPI4: Conn_01x01, Connector_PinSocket_2.00mm:PinSocket_1x01_P2.00mm_Vertical, B.Cu at (92.2, 81.0)
- added ULPI5: Conn_01x01, Connector_PinSocket_2.00mm:PinSocket_1x01_P2.00mm_Vertical, B.Cu at (98.2, 85.3)
- added ULPI6: Conn_01x01, Connector_PinSocket_2.00mm:PinSocket_1x01_P2.00mm_Vertical, B.Cu at (96.8, 78.9)
- added ULPI7: Conn_01x01, Connector_PinSocket_2.00mm:PinSocket_1x01_P2.00mm_Vertical, B.Cu at (103.5, 86.9)
- added ULPI8: Conn_01x01, Connector_PinSocket_2.00mm:PinSocket_1x01_P2.00mm_Vertical, B.Cu at (112.5, 83.6)
- added ULPI9: Conn_01x01, Connector_PinSocket_2.00mm:PinSocket_1x01_P2.00mm_Vertical, B.Cu at (107.7, 86.9)
- added USB1: USB_C_Receptacle_USB2.0, Connector_USB:USB_C_Receptacle_Palconn_UTC16-G, F.Cu at (44.5, 83.3)
- moved J3 22.1 mm to (56.9, 103.9)
- renumbered J1 to J2, J2 to J3
Connections:
- DATA1 pad 1: (no net) -> /ZYNQ_
- DATA1 pad 2: (no net) -> /ZYNQ_
- DATA1 pad 3: (no net) -> /ZYNQ_
- DATA1 pad 4: (no net) -> /ZYNQ_
- DATA2 pad 1: (no net) -> /ZYNQ_
- DATA2 pad 10: (no net) -> /ZYNQ_
- DATA2 pad 12: (no net) -> /ZYNQ_
- DATA2 pad 13: (no net) -> /ZYNQ_
- DATA2 pad 14: (no net) -> /ZYNQ_
- DATA2 pad 15: (no net) -> /ZYNQ_
- DATA2 pad 16: (no net) -> /ZYNQ_
- DATA2 pad 2: (no net) -> /ZYNQ_
- DATA2 pad 3: (no net) -> /ZYNQ_
- DATA2 pad 4: (no net) -> /ZYNQ_
- DATA2 pad 5: (no net) -> /ZYNQ_
- DATA2 pad 6: (no net) -> /ZYNQ_
- DATA2 pad 7: (no net) -> /ZYNQ_
- DATA2 pad 8: (no net) -> /ZYNQ_
- DATA3 pad 1: (no net) -> /ZYNQ_
- DATA3 pad 10: (no net) -> /ZYNQ_
- DATA3 pad 12: (no net) -> /ZYNQ_
- DATA3 pad 13: (no net) -> /ZYNQ_
- DATA3 pad 14: (no net) -> /ZYNQ_
- DATA3 pad 15: (no net) -> /ZYNQ_
- DATA3 pad 16: (no net) -> /ZYNQ_
- DATA3 pad 2: (no net) -> /ZYNQ_
- DATA3 pad 3: (no net) -> /ZYNQ_
- DATA3 pad 4: (no net) -> /ZYNQ_
- DATA3 pad 5: (no net) -> /ZYNQ_
- DATA3 pad 6: (no net) -> /ZYNQ_
- DATA3 pad 7: (no net) -> /ZYNQ_
- DATA3 pad 8: (no net) -> /ZYNQ_
